File: beerpimax.kicad_sch (KiCad schematic)
At the start: 4 parts, among them J1 Raspberry_Pi_2_3, J2 SSR Terminal, U1 MAX31865, U2 MAX31865

Commit message: board layout done
Parts:
- added FID1, FID2, FID3: Fiducial, Fiducial:Fiducial_1mm_Mask2mm, symbol Mechanical:Fiducial
- added MH1, MH2, MH3, MH4: M3, MountingHole:MountingHole_3.2mm_M3_Pad_Via, symbol Mechanical:MountingHole_Pad
- J1: renamed from J2; now left out of the parts list
- J2: renamed from J1; now left out of the parts list
- U1, U2: now left out of the parts list
Connections:
- net GND: now also MH1.1, MH2.1, MH3.1, MH4.1
- net SSRGPIO18: now reaches J1.1 (Pin_1), J2.12 (GPIO18/PWM0)
- net SPIGPIO8: now reaches J2.13 (GPIO27)
- net SPIGPIO8: now also U2.7 (CS)
- net SPIGPIO7: now reaches J2.15 (GPIO22)
- net SPIGPIO7: now also U1.7 (CS)
- net GPIO7: no longer names the net of J2.26 (~{CE1}/GPIO7)
- net GPIO7: no longer U1.7 (CS)
- net GPIO8: no longer names the net of J2.24 (~{CE0}/GPIO8)
- net GPIO8: no longer U2.7 (CS)
- net MISO renamed SPIMISO
- net MOSI renamed SPIMOSI
- net SCLK renamed SPISCLK
Other:
- note added: "AC SSR Terminal"
- note added: "MAX31865 RTC probe drivers"
- note added: "RPI Connector"
